File: Robi_I/kicad/RobiV4.kicad_pcb (KiCad board)
At the start: 2 copper layers, 67.7 x 95.3 mm, 28 parts, among them T1 Q_NPN_EBC, T1-B LP_rund, T2 Q_NPN_EBC, T2-B LP_rund, U1 NE555P, U2 BAT_HLD_SMD

Commit message: V 20.06.2024
Connections:
- T1 pad 1: Net-(Q1-C) -> Net-(D1-K)
- T2 pad 1: Net-(Q2-C) -> Net-(D1-A)
- T2 pad 3: Net-(D1-A) -> Net-(Q2-C)
Routing:
- net Net-(Q1-C): track 57.6 -> 51.6 mm, vias 1 -> 0
- net Net-(Q2-C): track 43.7 -> 46.4 mm
- net Net-(D1-K): track 146.8 -> 147.3 mm, vias 2 -> 3
- net Net-(D3-A): track 80.8 -> 80.7 mm, vias 0 -> 1
Other:
- board text added: "KHF 06.2024"
- board text removed: "KHF 01.2024"

Commit message: V 03082024
Parts:
- T1, T2: moved to F.Cu
- moved T2 4.90 mm to (158.9, 83.3), turned to 180 degrees
- moved T1 4.22 mm to (132.1, 86.8), turned to 180 degrees
Connections:
- T1-B pad 1: Net-(T1-B) -> Net-(Q1-B)
Routing:
- net Net-(D1-K): track 147.3 -> 182.7 mm, vias 3 -> 2
- net Net-(Q1-C): track 51.6 -> 57.8 mm
- net Net-(T1-B): track 5.31 -> 0.00 mm
- net Net-(Q2-C): track 46.4 -> 50.3 mm
- net Net-(Q1-B): track 27.9 -> 30.0 mm
Other:
- board text added: "KHF 08.2024"
- board text removed: "KHF 06.2024"
