File: Kuh/kicad/Cow.kicad_pcb (KiCad board)
At the start: 2 copper layers, 94.2 x 99.9 mm, 26 parts, among them Q1 BC558, Q2 BC558, U1 NE555P, U2 BAT_HLD_SMD

Commit message: V 10092024
Routing:
- net Net-(D3-A): track 31.5 -> 35.5 mm
- net Net-(D3-K): track 64.7 -> 63.8 mm
Changed lines of the file:
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@@
   (segment (start 153.44 119.16) (end 156.12 119.16) (width 0.25) (layer "F.Cu") (net 1))
   (segment (start 156.12 119.16) (end 154.56 119.16) (width 0.25) (layer "B.Cu") (net 1))
+  (segment (start 156.16 130.45) (end 156.16 132.05) (width 0.25) (layer "B.Cu") (net 1))
   (segment (start 157.8 119.16) (end 157.8 128.81) (width 0.25) (layer "B.Cu") (net 1))
   (segment (start 148.41 139.8) (end 156.16 132.05) (width 0.25) (layer "B.Cu") (net 1))
-  (segment (start 156.16 131.81) (end 156.16 132.66) (width 0.25) (layer "B.Cu") (net 1))
   (segment (start 152.02 121.7) (end 148.5 121.7) (width 0.25) (layer "B.Cu") (net 1))
-  (segment (start 156.16 132.05) (end 156.16 131.81) (width 0.25) (layer "B.Cu") (net 1))
   (segment (start 154.56 119.16) (end 152.02 121.7) (width 0.25) (layer "B.Cu") (net 1))
   (segment (start 156.12 119.16) (end 157.8 119.16) (width 0.25) (layer "B.Cu") (net 1))
   (segment (start 148.5 121.7) (end 144.69 121.7) (width 0.25) (layer "B.Cu") (net 1))
   (segment (start 144.69 121.7) (end 143.26 123.13) (width 0.25) (layer "B.Cu") (net 1))
-  (segment (start 156.16 130.45) (end 156.16 131.81) (width 0.25) (layer "B.Cu") (net 1))
   (segment (start 157.8 128.81) (end 156.16 130.45) (width 0.25) (layer "B.Cu") (net 1))
   (segment (start 138.58 110.98) (end 140.37 112.77) (width 0.25) (layer "F.Cu") (net 2))
@@
   (segment (start 148.54 130.45) (end 136.28 130.45) (width 0.25) (layer "B.Cu") (net 4))
   (segment (start 136.28 130.36) (end 133.1 127.18) (width 0.25) (layer "B.Cu") (net 4))
+  (segment (start 133.1 123.13) (end 133.1 127.18) (width 0.25) (layer "B.Cu") (net 4))
   (segment (start 123.13 98.81361) (end 123.13 102.45) (width 0.25) (layer "F.Cu") (net 5))
   (segment (start 141.19 110.98) (end 137.14 106.93) (width 0.25) (layer "F.Cu") (net 5))
