File: Rocket/kicad/Rocket.kicad_pcb (KiCad board)
At the start: 2 copper layers, 135.2 x 112.1 mm, 35 parts, among them Q1 Q_NPN_EBC, Q2 Q_NPN_EBC, U1 NE555P, U2 BAT_HLD_SMD

Commit message: V03012026
Parts:
- removed the G*** at (131.6, 96.3) (x7)
- removed the G*** at (136.6, 104.1) (x6)
- removed the G*** at (136.4, 104.1) (x6)
- added G*** (x6): LOGO, LOGO, F.Cu at (99.6, 105.9)
- added G*** (x6): LOGO, LOGO, F.Cu at (94.6, 98.1)
- added G*** (x6): LOGO, LOGO, F.Cu at (99.4, 105.9)
- added G*** (x7): LOGO, LOGO, F.Cu at (108.0, 101.2)
- moved Q2 37.1 mm to (123.9, 133.0)
- moved U2 37.1 mm to (115.3, 58.4)
- moved Q1 37.1 mm to (127.1, 122.9)
- moved R3 37.1 mm to (90.1, 134.8)
- moved R4 37.1 mm to (90.1, 130.7)
- moved R5 37.1 mm to (90.1, 126.7)
- moved R6 37.1 mm to (90.1, 122.6)
- moved R7 37.1 mm to (90.1, 118.6)
- moved R8 37.1 mm to (90.1, 114.5)
- moved S1 37.1 mm to (135.6, 112.6)
- moved U1 37.1 mm to (110.6, 114.7)
- moved C1 37.1 mm to (112.6, 123.2)
- moved D3 37.1 mm to (110.6, 103.3)
- moved G*** 37.0 mm to (121.9, 105.5)
- moved D1 35.5 mm to (126.9, 79.1)
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Routing:
- net Net-(D1-A): track 97.1 -> 95.2 mm
- net Net-(D1-K): track 168.0 -> 169.6 mm
Other:
- board size 135.2 x 112.1 mm -> 120.2 x 99.7 mm

Commit message: V09012026
Routing:
- net Net-(D3-K): track 108.9 -> 131.2 mm
- net Net-(Q2-C): track 36.8 -> 33.0 mm
- net Net-(Q1-C): track 61.3 -> 59.9 mm
Other:
- board text added: "KHF 01.2026"
- board text removed: "KHF 12.2025"
Changed lines of the file:
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@@
 		(layer "Edge.Cuts")
 	)
-	(gr_text "KHF 12.2025"
+	(gr_text "KHF 01.2026"
 		(at 121.693 72.315 0)
 		(layer "B.Cu")
@@
 		)
 	)
-	(gr_text "KHF 12.2025"
+	(gr_text "KHF 01.2026"
 		(at 121.693 72.315 0)
 		(layer "B.Mask")
@@
 	)
 	(segment
+		(start 90.133 134.765)
+		(end 94.9 129.998)
+		(width 0.25)
+		(layer "F.Cu")
+		(net 1)
+	)
+	(segment
 		(start 116.8465 109.6685)
 		(end 112.793 105.615)
@@
 	)
 	(segment
+		(start 94.9 119.65)
+		(end 94.85 119.65)
+		(width 0.25)
+		(layer "F.Cu")
+		(net 1)
+	)
+	(segment
 		(start 118.2469 109.6685)
 		(end 116.8465 109.6685)
@@
 	)
 	(segment
+		(start 93.765 118.565)
+		(end 90.133 118.565)
+		(width 0.25)
+		(layer "F.Cu")
+		(net 1)
+	)
+	(segment
 		(start 126.793 99.615)
 		(end 126.793 106.115)
@@
 	)
 	(segment
+		(start 94.85 119.65)
+		(end 93.765 118.565)
+		(width 0.25)
+		(layer "F.Cu")
+		(net 1)
+	)
+	(segment
 		(start 112.793 105.615)
 		(end 86.793 105.615)
@@
 	)
 	(segment
+		(start 94.9 129.998)
+		(end 94.9 119.65)
+		(width 0.25)
+		(layer "F.Cu")
+		(net 1)
+	)
+	(segment
 		(start 123.2395 109.6685)
 		(end 118.2469 109.6685)
@@
 	)
 	(segment
+		(start 114.25 130.95)
+		(end 124.3 130.95)
+		(width 0.25)
+		(layer "F.Cu")
+		(net 6)
+	)
+	(segment
+		(start 126.316192 133.033808)
+		(end 128.933 133.033808)
+		(width 0.25)
+		(layer "F.Cu")
+		(net 6)
+	)
+	(segment
+		(start 126.3 133.05)
+		(end 126.316192 133.033808)
+		(width 0.25)
+		(layer "F.Cu")
+		(net 6)
+	)
+	(segment
+		(start 124.3 130.95)
+		(end 126.3 132.95)
+		(width 0.25)
+		(layer "F.Cu")
+		(net 6)
+	)
+	(segment
 		(start 100.293 122.615)
-		(end 103.793 122.615)
+		(end 105.915 122.615)
 		(width 0.25)
 		(layer "F.Cu")
@@
 	)
 	(segment
-		(start 126.793 136.615)
-		(end 128.933 134.475)
+		(start 126.3 132.95)
+		(end 126.3 133.05)
 		(width 0.25)
 		(layer "F.Cu")
@@
 	)
 	(segment
-		(start 128.933 134.475)
-		(end 128.933 133.033808)
+		(start 105.915 122.615)
+		(end 114.25 130.95)
 		(width 0.25)
 		(layer "F.Cu")
@@
 	)
 	(segment
-		(start 117.793 136.615)
-		(end 126.793 136.615)
-		(width 0.25)
-		(layer "F.Cu")
-		(net 6)
-	)
-	(segment
-		(start 103.793 122.615)
-		(end 117.793 136.615)
-		(width 0.25)
-		(layer "F.Cu")
-		(net 6)
+		(start 131.293 137.307)
+		(end 131.25 137.35)
+		(width 0.25)
+		(layer "F.Cu")
+		(net 7)
+	)
+	(segment
+		(start 105.793 133.943)
+		(end 105.793 127.615)
+		(width 0.25)
+		(layer "F.Cu")
+		(net 7)
+	)
+	(segment
+		(start 131.293 132.115)
+		(end 131.293 137.307)
+		(width 0.25)
+		(layer "F.Cu")
+		(net 7)
+	)
+	(segment
+		(start 123.45 137.35)
+		(end 122.3 136.2)
+		(width 0.25)
+		(layer "F.Cu")
+		(net 7)
+	)
+	(segment
+		(start 122.3 136.2)
+		(end 108.05 136.2)
+		(width 0.25)
+		(layer "F.Cu")
+		(net 7)
+	)
+	(segment
+		(start 131.25 137.35)
+		(end 123.45 137.35)
+		(width 0.25)
+		(layer "F.Cu")
+		(net 7)
+	)
+	(segment
+		(start 105.793 127.615)
+		(end 104.843 126.665)
+		(width 0.25)
+		(layer "F.Cu")
+		(net 7)
 	)
 	(segment
@@
 	)
 	(segment
-		(start 131.293 139.115)
-		(end 112.793 139.115)
-		(width 0.25)
-		(layer "F.Cu")
-		(net 7)
-	)
-	(segment
-		(start 112.793 139.115)
-		(end 105.793 132.115)
-		(width 0.25)
-		(layer "F.Cu")
-		(net 7)
-	)
-	(segment
-		(start 105.793 127.615)
-		(end 104.843 126.665)
-		(width 0.25)
-		(layer "F.Cu")
-		(net 7)
-	)
-	(segment
-		(start 131.293 132.115)
-		(end 131.293 139.115)
+		(start 104.843 126.665)
+		(end 100.293 126.665)
 		(width 0.25)
 		(layer "F.Cu")
@@
 	)
 	(segment
-		(start 104.843 126.665)
-		(end 100.293 126.665)
-		(width 0.25)
-		(layer "F.Cu")
-		(net 7)
-	)
-	(segment
-		(start 105.793 132.115)
-		(end 105.793 127.615)
-		(width 0.25)
-		(layer "F.Cu")
+		(start 108.05 136.2)
+		(end 105.793 133.943)
+		(width 0.25)
+		(layer "F.Cu")
