File: Alligator/kicad/Alligator.kicad_pcb (KiCad board)
At the start: 2 copper layers, 140.6 x 93 mm, 24 parts, among them Q1 Q_NPN_EBC, Q2 Q_NPN_EBC, U1 NE555P, U2 BAT_HLD_SMD

Commit message: V23012026
Parts:
- Q1, Q2: moved to F.Cu
- moved Q2 5.20 mm to (120.6, 114.3), turned to 90 degrees
- moved Q1 5.00 mm to (111.9, 114.0), turned to 90 degrees
- moved U2 2.20 mm to (162.2, 99.3)
Routing:
- net Net-(D1-A): track 62.6 -> 92.4 mm
- net Net-(D1-K): track 223.3 -> 247.8 mm
- net Net-(S1-A-Pad1): track 65.9 -> 67.3 mm
- net Net-(Q1-C): track 32.4 -> 33.6 mm
- net Net-(Q2-C): track 19.6 -> 20.7 mm
Other:
- board text added: "KHF 01.2026"
- board text added: "USB-C"
- board text removed: "KHF 12.2025"
