File: Seegeist/kicad/Seegeist.kicad_pcb (KiCad board)
At the start: 2 copper layers, 93.8 x 84.9 mm, 32 parts, among them Q1 Q_NPN_EBC, Q2 Q_NPN_EBC, U2 BAT_HLD_SMD

Commit message: V25012026
Parts:
- moved G*** 50.2 mm to (143.1, 148.0)
- renumbered R5 to R3, R6 to R4, R7 to R5, R8 to R6
Other:
- board text added: "${REFERENCE}"
- board text added: "R1"
- board text added: "R2"
- board text removed: "KHF 11.2025"
Changed lines of the file:
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@@
 	(footprint "!Goody:ob-logo_B.SilkS"
 		(layer "F.Cu")
-		(at 141.95 97.85)
+		(at 143.1 148)
 		(descr "Oberlab-Logo B.SilkS")
 		(property "Reference" "G***"
@@
 			(at 1.25 -4.4 0)
 			(layer "B.Fab")
+			(hide yes)
 			(effects
 				(font
@@
 			(layer "B.SilkS")
 		)
-		(fp_line
-			(start -3.185 0.315)
-			(end -3.185 -0.315)
-			(stroke
-				(width 0.12)
-				(type solid)
-			)
-			(layer "B.SilkS")
-		)
-		(fp_line
-			(start -3.5 0)
-			(end -2.87 0)
-			(stroke
-				(width 0.12)
-				(type solid)
-			)
-			(layer "B.SilkS")
-		)
 		(fp_circle
 			(center 1.25 0)
@@
 		(descr "Resistor, Axial_DIN0207 series, Axial, Horizontal, pin pitch=10.16mm, 0.25W = 1/4W, length*diameter=6.3*2.5mm^2, http://cdn-reichelt.de/documents/datenblatt/B400/1_4W%23YAG.pdf")
 		(tags "Resistor Axial_DIN0207 series Axial Horizontal pin pitch 10.16mm 0.25W = 1/4W length 6.3mm diameter 2.5mm")
-		(property "Reference" "R7"
-			(at 5.08 0.014 0)
+		(property "Reference" "R5"
+			(at 4.953 -0.0114 0)
 			(layer "B.SilkS")
 			(effects
@@
 			(layer "B.Fab")
 		)
-		(fp_text user "${REFERENCE}"
-			(at 5.08 0 0)
-			(layer "B.Fab")
-			(effects
-				(font
-					(size 1 1)
-					(thickness 0.15)
-				)
-				(justify mirror)
-			)
-		)
 		(pad "1" thru_hole circle
 			(at 0 0 180)
@@
 			(layer "B.Fab")
 		)
-		(fp_text user "${REFERENCE}"
-			(at 5.08 0 0)
-			(layer "B.SilkS")
-			(effects
-				(font
-					(size 1 1)
-					(thickness 0.15)
-				)
-				(justify mirror)
-			)
-		)
 		(pad "1" thru_hole circle
 			(at 0 0 180)
@@
 			(layer "B.Fab")
 		)
-		(fp_text user "R3"
-			(at 4.826 -0.057 0)
-			(layer "B.SilkS")
-			(effects
-				(font
-					(size 1 1)
-					(thickness 0.15)
-				)
-				(justify mirror)
-			)
-		)
 		(pad "1" thru_hole circle
 			(at 0 0 180)
@@
 		(descr "Resistor, Axial_DIN0207 series, Axial, Horizontal, pin pitch=10.16mm, 0.25W = 1/4W, length*diameter=6.3*2.5mm^2, http://cdn-reichelt.de/documents/datenblatt/B400/1_4W%23YAG.pdf")
 		(tags "Resistor Axial_DIN0207 series Axial Horizontal pin pitch 10.16mm 0.25W = 1/4W length 6.3mm diameter 2.5mm")
-		(property "Reference" "R5"
-			(at 4.953 0.042 0)
+		(property "Reference" "R3"
+			(at 4.953 -0.0342 0)
 			(layer "B.SilkS")
 			(effects
@@
 			(layer "B.Fab")
 		)
-		(fp_text user "${REFERENCE}"
-			(at 5.08 0 0)
-			(layer "B.Fab")
-			(effects
-				(font
-					(size 1 1)
-					(thickness 0.15)
-				)
-				(justify mirror)
-			)
-		)
 		(pad "1" thru_hole circle
 			(at 0 0 180)
@@
 		(descr "Resistor, Axial_DIN0207 series, Axial, Horizontal, pin pitch=10.16mm, 0.25W = 1/4W, length*diameter=6.3*2.5mm^2, http://cdn-reichelt.de/documents/datenblatt/B400/1_4W%23YAG.pdf")
 		(tags "Resistor Axial_DIN0207 series Axial Horizontal pin pitch 10.16mm 0.25W = 1/4W length 6.3mm diameter 2.5mm")
-		(property "Reference" "R8"
+		(property "Reference" "R6"
 			(at 4.953 0 0)
 			(layer "B.SilkS")
@@
 			(layer "B.Fab")
 		)
-		(fp_text user "${REFERENCE}"
-			(at 5.08 0 0)
-			(layer "B.Fab")
-			(effects
-				(font
-					(size 1 1)
-					(thickness 0.15)
-				)
-				(justify mirror)
-			)
-		)
 		(pad "1" thru_hole circle
 			(at 0 0 180)
@@
 		(descr "Resistor, Axial_DIN0207 series, Axial, Horizontal, pin pitch=10.16mm, 0.25W = 1/4W, length*diameter=6.3*2.5mm^2, http://cdn-reichelt.de/documents/datenblatt/B400/1_4W%23YAG.pdf")
 		(tags "Resistor Axial_DIN0207 series Axial Horizontal pin pitch 10.16mm 0.25W = 1/4W length 6.3mm diameter 2.5mm")
-		(property "Reference" "R6"
-			(at 5.08 0.028 0)
+		(property "Reference" "R4"
+			(at 4.953 -0.0228 0)
 			(layer "B.SilkS")
 			(effects
@@
 			(layer "B.Fab")
 		)
-		(fp_text user "${REFERENCE}"
-			(at 5.08 0 0)
-			(layer "B.Fab")
-			(effects
-				(font
-					(size 1 1)
-					(thickness 0.15)
-				)
-				(justify mirror)
-			)
-		)
 		(pad "1" thru_hole circle
 			(at 0 0 180)
@@
 	)
 	(gr_text "KHF 01.2026"
-		(at 142.2 65.55 0)
+		(at 141.9 137.2 0)
 		(layer "B.Cu")
 		(effects
@@
 		)
 	)
-	(gr_text "KHF 11.2025"
-		(at 247.519 148.95 0)
-		(layer "B.Mask")
-		(effects
-			(font
-				(size 1 1)
-				(thickness 0.15)
-			)
-			(justify left bottom mirror)
-		)
-	)
 	(gr_text "KHF 01.2026"
-		(at 142.2 65.55 0)
+		(at 141.9 137.2 0)
 		(layer "B.Mask")
 		(effects
@@
 		)
 	)
+	(gr_text "R2"
+		(at 115.657 92.5456 0)
+		(layer "B.SilkS")
+		(effects
+			(font
+				(size 1 1)
+				(thickness 0.15)
+			)
+			(justify mirror)
+		)
+	)
+	(gr_text "R1"
+		(at 115.657 88.507 0)
+		(layer "B.SilkS")
+		(effects
+			(font
+				(size 1 1)
+				(thickness 0.15)
+			)
+			(justify mirror)
+		)
+	)
 	(gr_text "1N4148"
 		(at 154.4 92.185 270)
@@
 	)
 	(gr_text "E"
-		(at 98.85 90.75 180)
+		(at 99.8 90.8 180)
 		(layer "B.SilkS")
 		(effects
@@
 				(thickness 0.15)
 			)
-			(justify left bottom mirror)
+			(justify left bottom)
 		)
 	)
@@
 		(effects
 			(font
+				(size 1 1)
+				(thickness 0.15)
+			)
+			(justify mirror)
+		)
+	)
+	(gr_text "${REFERENCE}"
+		(at 115.53 100.6 0)
+		(layer "B.Fab")
+		(effects
+			(font
